File: mssculpt.kicad_pcb (KiCad board)
At the start: 2 copper layers, 47.5 x 40 mm, 9 parts, among them J1 keyboard, J2 debug, J3 power, U1 E73-2G4M04S-52832

Commit message: final optimizations
Routing:
- net GND: track 0.00 -> 1.00 mm, vias 112 -> 114
Other:
- board text added: "github.com/M1cha/microsoft_sculpt_hardware"
- board text added: "v1.0"
