File: mssculpt.sch (KiCad schematic (older format))
At the start: 6 parts, among them J1 keyboard, J2 debug, J3 power, U1 E73-2G4M04S-52832

Commit message: backup
Parts:
- C1: value C_Small -> 100n
- R1: value R -> 4K7
Changed lines of the file:
@@
 P 10050 5500
 F 0 "R1" H 10120 5546 50  0000 L CNN
-F 1 "R" H 10120 5455 50  0000 L CNN
+F 1 "4K7" H 10120 5455 50  0000 L CNN
 F 2 "Resistor_SMD:R_0805_2012Metric_Pad1.20x1.40mm_HandSolder" V 9980 5500 50  0001 C CNN
 F 3 "~" H 10050 5500 50  0001 C CNN
@@
 P 5650 1950
 F 0 "C1" V 5879 1950 50  0000 C CNN
-F 1 "C_Small" V 5788 1950 50  0000 C CNN
+F 1 "100n" V 5788 1950 50  0000 C CNN
 F 2 "Capacitor_SMD:C_0805_2012Metric_Pad1.18x1.45mm_HandSolder" H 5650 1950 50  0001 C CNN
 F 3 "~" H 5650 1950 50  0001 C CNN
